File: usb-4-uart-FT4232H.kicad_pcb (KiCad board)
At the start: 2 copper layers, 20 x 50 mm, 28 parts, among them J1 Conn_02x05_Odd_Even, U1 FT4232H, Y1 12MHz

Commit message: updated silkscreen
Other:
- board text added: "USB to 4x UART Luis Alvarez 00.01.00"
Changed lines of the file:
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@@
+		)
+	)
+	(gr_text "USB to 4x UART\nLuis Alvarez\n00.01.00"
+		(at 30.1 37.4 0)
+		(layer "B.SilkS")
+		(effects
+			(font
+				(size 1 1)
+				(thickness 0.1)
+			)
+			(justify bottom mirror)
 		)
 	)
